File: electronics/drake_electronics/drake_electronics.kicad_sch (KiCad schematic)
At the start: 2 parts

Commit message: basic schematic
Parts:
- added P?: Conn_WallPlug_Earth, symbol Connector:Conn_WallPlug_Earth
- added PS? (x2): VTX-214-015-124, Converter_ACDC:Converter_ACDC_Vigortronix_VTX-214-015-1xx_THT, symbol Converter_ACDC:VTX-214-015-124
Connections:
- new net: P?.2 (AC_N), PS?.2 (N), PS?.2 (N)
- new net: P?.1 (AC_P), PS?.3 (L), PS?.3 (L)
Other:
- moved on the sheet: M?, U?
Changed lines of the file:
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@@
 (kicad_sch (version 20211123) (generator eeschema)
-  (paper "A4")
-  (wire (pts (xy 159.385 40.64) (xy 177.165 40.64))
-    (stroke (width 0) (type default) (color 0 0 0 0))
-  )
-  (wire (pts (xy 151.13 50.165) (xy 164.465 50.165))
-    (stroke (width 0) (type default) (color 0 0 0 0))
-  )
-  (wire (pts (xy 151.13 47.625) (xy 161.925 47.625))
-    (stroke (width 0) (type default) (color 0 0 0 0))
-  )
-  (wire (pts (xy 161.925 38.1) (xy 182.245 38.1))
-    (stroke (width 0) (type default) (color 0 0 0 0))
-  )
-  (wire (pts (xy 177.165 40.64) (xy 177.165 42.545))
-    (stroke (width 0) (type default) (color 0 0 0 0))
-  )
-  (wire (pts (xy 182.245 38.1) (xy 182.245 42.545))
-    (stroke (width 0) (type default) (color 0 0 0 0))
-  )
-  (wire (pts (xy 161.925 47.625) (xy 161.925 38.1))
-    (stroke (width 0) (type default) (color 0 0 0 0))
-  )
-  (wire (pts (xy 164.465 50.165) (xy 164.465 47.625))
-    (stroke (width 0) (type default) (color 0 0 0 0))
-  )
-  (wire (pts (xy 159.385 45.085) (xy 159.385 40.64))
-    (stroke (width 0) (type default) (color 0 0 0 0))
-  )
-  (wire (pts (xy 151.13 45.085) (xy 159.385 45.085))
-    (stroke (width 0) (type default) (color 0 0 0 0))
-  )
-  (wire (pts (xy 164.465 47.625) (xy 172.085 47.625))
-    (stroke (width 0) (type default) (color 0 0 0 0))
-  )
-  (wire (pts (xy 151.13 52.705) (xy 172.085 52.705))
-    (stroke (width 0) (type default) (color 0 0 0 0))
-  )
-  (symbol (lib_id "Motor:Stepper_Motor_bipolar") (at 179.705 50.165 0) (unit 1)
+  (paper "A3")
+  (junction (at 72.39 34.29) (diameter 0) (color 0 0 0 0)
+  )
+  (junction (at 67.31 37.465) (diameter 0) (color 0 0 0 0)
+  )
+  (wire (pts (xy 228.6 69.85) (xy 246.38 69.85))
+    (stroke (width 0) (type default) (color 0 0 0 0))
+  )
+  (wire (pts (xy 220.345 79.375) (xy 233.68 79.375))
+    (stroke (width 0) (type default) (color 0 0 0 0))
+  )
+  (wire (pts (xy 67.31 52.705) (xy 108.585 52.705))
+    (stroke (width 0) (type default) (color 0 0 0 0))
+  )
+  (wire (pts (xy 67.31 34.29) (xy 67.31 37.465))
+    (stroke (width 0) (type default) (color 0 0 0 0))
+  )
+  (wire (pts (xy 220.345 76.835) (xy 231.14 76.835))
+    (stroke (width 0) (type default) (color 0 0 0 0))
+  )
+  (wire (pts (xy 67.31 37.465) (xy 67.31 52.705))
+    (stroke (width 0) (type default) (color 0 0 0 0))
+  )
+  (wire (pts (xy 231.14 67.31) (xy 251.46 67.31))
+    (stroke (width 0) (type default) (color 0 0 0 0))
+  )
+  (wire (pts (xy 72.39 34.29) (xy 108.585 34.29))
+    (stroke (width 0) (type default) (color 0 0 0 0))
+  )
+  (wire (pts (xy 246.38 69.85) (xy 246.38 71.755))
+    (stroke (width 0) (type default) (color 0 0 0 0))
+  )
+  (wire (pts (xy 251.46 67.31) (xy 251.46 71.755))
+    (stroke (width 0) (type default) (color 0 0 0 0))
+  )
+  (wire (pts (xy 67.31 37.465) (xy 108.585 37.465))
+    (stroke (width 0) (type default) (color 0 0 0 0))
+  )
+  (wire (pts (xy 231.14 76.835) (xy 231.14 67.31))
+    (stroke (width 0) (type default) (color 0 0 0 0))
+  )
+  (wire (pts (xy 72.39 33.655) (xy 72.39 34.29))
+    (stroke (width 0) (type default) (color 0 0 0 0))
+  )
+  (wire (pts (xy 233.68 79.375) (xy 233.68 76.835))
+    (stroke (width 0) (type default) (color 0 0 0 0))
+  )
+  (wire (pts (xy 228.6 74.295) (xy 228.6 69.85))
+    (stroke (width 0) (type default) (color 0 0 0 0))
+  )
+  (wire (pts (xy 72.39 47.625) (xy 108.585 47.625))
+    (stroke (width 0) (type default) (color 0 0 0 0))
+  )
+  (wire (pts (xy 108.585 34.29) (xy 108.585 32.385))
+    (stroke (width 0) (type default) (color 0 0 0 0))
+  )
+  (wire (pts (xy 72.39 34.29) (xy 72.39 47.625))
+    (stroke (width 0) (type default) (color 0 0 0 0))
+  )
+  (wire (pts (xy 220.345 74.295) (xy 228.6 74.295))
+    (stroke (width 0) (type default) (color 0 0 0 0))
+  )
+  (wire (pts (xy 233.68 76.835) (xy 241.3 76.835))
+    (stroke (width 0) (type default) (color 0 0 0 0))
+  )
+  (wire (pts (xy 220.345 81.915) (xy 241.3 81.915))
+    (stroke (width 0) (type default) (color 0 0 0 0))
+  )
+  (symbol (lib_id "Motor:Stepper_Motor_bipolar") (at 248.92 79.375 0) (unit 1)
     (in_bom yes) (on_board yes) (fields_autoplaced)
-    (property "Reference" "M?" (id 0) (at 184.785 48.044 0)
-      (effects (font (size 1.27 1.27)) (justify left))
-    )
-    (property "Value" "Stepper_Motor_bipolar" (id 1) (at 184.785 50.584 0)
-      (effects (font (size 1.27 1.27)) (justify left))
-    )
-    (property "Footprint" "" (id 2) (at 179.959 50.419 0)
-      (effects (font (size 1.27 1.27)) hide)
-    )
-    (property "Datasheet" "http://www.infineon.com/dgdl/Application-Note-TLE8110EE_driving_UniPolarStepperMotor_V1.1.pdf?fileId=db3a30431be39b97011be5d0aa0a00b0" (id 3) (at 179.959 50.419 0)
-      (effects (font (size 1.27 1.27)) hide)
-    )
-    (pin "1")
-    (pin "2")
-    (pin "3")
-    (pin "4")
-  )
-  (symbol (lib_id "Driver_Motor:SYRD_MK1") (at 133.35 103.505 0) (unit 1)
+    (property "Reference" "M?" (id 0) (at 254 77.254 0)
+      (effects (font (size 1.27 1.27)) (justify left))
+    )
+    (property "Value" "Stepper_Motor_bipolar" (id 1) (at 254 79.794 0)
+      (effects (font (size 1.27 1.27)) (justify left))
+    )
+    (property "Footprint" "" (id 2) (at 249.174 79.629 0)
+      (effects (font (size 1.27 1.27)) hide)
+    )
+    (property "Datasheet" "http://www.infineon.com/dgdl/Application-Note-TLE8110EE_driving_UniPolarStepperMotor_V1.1.pdf?fileId=db3a30431be39b97011be5d0aa0a00b0" (id 3) (at 249.174 79.629 0)
+      (effects (font (size 1.27 1.27)) hide)
+    )
+    (pin "1")
+    (pin "2")
+    (pin "3")
+    (pin "4")
+  )
+  (symbol (lib_id "Converter_ACDC:VTX-214-015-124") (at 118.745 34.925 0) (unit 1)
+    (in_bom yes) (on_board yes)
+    (property "Reference" "PS?" (id 0) (at 118.745 27.94 0))
+    (property "Value" "VTX-214-015-124" (id 1) (at 118.745 26.67 0)
+      (effects (font (size 1.27 1.27)) hide)
+    )
+    (property "Footprint" "Converter_ACDC:Converter_ACDC_Vigortronix_VTX-214-015-1xx_THT" (id 2) (at 118.745 23.495 0)
+      (effects (font (size 1.27 1.27)) hide)
+    )
+    (property "Datasheet" "http://www.vigortronix.com/15WattSMPSPCBModuleAC-DC" (id 3) (at 146.685 55.245 0)
+      (effects (font (size 1.27 1.27)) hide)
+    )
+    (pin "1")
+    (pin "2")
+    (pin "3")
+    (pin "4")
+    (pin "5")
+  )
+  (symbol (lib_id "Converter_ACDC:VTX-214-015-124") (at 118.745 50.165 0) (unit 1)
+    (in_bom yes) (on_board yes)
+    (property "Reference" "PS?" (id 0) (at 118.745 43.815 0))
+    (property "Value" "VTX-214-015-124" (id 1) (at 118.745 41.91 0)
+      (effects (font (size 1.27 1.27)) hide)
+    )
+    (property "Footprint" "Converter_ACDC:Converter_ACDC_Vigortronix_VTX-214-015-1xx_THT" (id 2) (at 118.745 38.735 0)
+      (effects (font (size 1.27 1.27)) hide)
+    )
+    (property "Datasheet" "http://www.vigortronix.com/15WattSMPSPCBModuleAC-DC" (id 3) (at 146.685 70.485 0)
+      (effects (font (size 1.27 1.27)) hide)
+    )
+    (pin "1")
+    (pin "2")
+    (pin "3")
+    (pin "4")
+    (pin "5")
+  )
+  (symbol (lib_id "Connector:Conn_WallPlug_Earth") (at 69.85 26.67 270) (unit 1)
     (in_bom yes) (on_board yes) (fields_autoplaced)
-    (property "Reference" "U?" (id 0) (at 135.3694 36.83 0)
-      (effects (font (size 1.27 1.27)) (justify left))
-    )
-    (property "Value" "SYRD_MK1" (id 1) (at 135.3694 39.37 0)
-      (effects (font (size 1.27 1.27)) (justify left))
-    )
-    (property "Footprint" "" (id 2) (at 133.35 102.235 0)
-      (effects (font (size 1.27 1.27)) hide)
-    )
-    (property "Datasheet" "" (id 3) (at 133.35 102.235 0)
+    (property "Reference" "P?" (id 0) (at 74.93 25.0062 90)
+      (effects (font (size 1.27 1.27)) (justify left))
+    )
+    (property "Value" "Conn_WallPlug_Earth" (id 1) (at 74.93 27.5462 90)
+      (effects (font (size 1.27 1.27)) (justify left))
+    )
+    (property "Footprint" "" (id 2) (at 69.85 36.83 0)
+      (effects (font (size 1.27 1.27)) hide)
+    )
+    (property "Datasheet" "~" (id 3) (at 69.85 36.83 0)
+      (effects (font (size 1.27 1.27)) hide)
+    )
+    (pin "1")
+    (pin "2")
+    (pin "3")
+  )
+  (symbol (lib_id "Driver_Motor:SYRD_MK1") (at 202.565 132.715 0) (unit 1)
+    (in_bom yes) (on_board yes) (fields_autoplaced)
+    (property "Reference" "U?" (id 0) (at 204.5844 66.04 0)
+      (effects (font (size 1.27 1.27)) (justify left))
+    )
+    (property "Value" "SYRD_MK1" (id 1) (at 204.5844 68.58 0)
+      (effects (font (size 1.27 1.27)) (justify left))
+    )
+    (property "Footprint" "" (id 2) (at 202.565 131.445 0)
+      (effects (font (size 1.27 1.27)) hide)
+    )
+    (property "Datasheet" "" (id 3) (at 202.565 131.445 0)
       (effects (font (size 1.27 1.27)) hide)
     )
@@
       (reference "M?") (unit 1) (value "Stepper_Motor_bipolar") (footprint "")
     )
+    (path "/b81acb8a-0382-4364-91db-dc21854abd4d"
+      (reference "P?") (unit 1) (value "Conn_WallPlug_Earth") (footprint "")
+    )
+    (path "/8b29c40a-a541-411b-ae4b-66b6732b7d62"
+      (reference "PS?") (unit 1) (value "VTX-214-015-124") (footprint "Converter_ACDC:Converter_ACDC_Vigortronix_VTX-214-015-1xx_THT")
+    )
+    (path "/ab482a78-25fb-454e-b3ed-18ba8bd0fc5e"
+      (reference "PS?") (unit 1) (value "VTX-214-015-124") (footprint "Converter_ACDC:Converter_ACDC_Vigortronix_VTX-214-015-1xx_THT")
+    )
     (path "/ce9bdf49-69fd-4f1a-b670-fdbdb97a8355"

Commit message: finsihed basic electronics
Parts:
- added CB1: CircuitBreaker_2P, symbol Device:CircuitBreaker_2P
- added J1: Conn_01x02_Female, symbol Connector:Conn_01x02_Female
- added J2: Conn_01x02_Male, symbol Connector:Conn_01x02_Male
- added J3: Raspberry_Pi_2_3, symbol Connector:Raspberry_Pi_2_3
- added M2, M3, M4: Stepper_Motor_bipolar, symbol Motor:Stepper_Motor_bipolar
- added M5: Motor_DC, symbol Motor:Motor_DC
- added SW1: SW_DPST, symbol Switch:SW_DPST
- added SW2, SW3: SW_Push_Lamp, symbol Switch:SW_Push_Lamp
- added SW4, SW5, SW6, SW7, SW8, SW9: SW_Push_Open, symbol Switch:SW_Push_Open
- added U2: A4950E, Package_SO:SOIC-8-1EP_3.9x4.9mm_P1.27mm_EP2.41x3.3mm, symbol Driver_Motor:A4950E
- gave numbers to parts that had none: 5
Connections:
- net at PS1.2 (N), PS2.2 (N): now also SW1.3; no longer P1.2 (AC_N)
- net at PS1.3 (L), PS2.3 (L): now also SW1.1; no longer P1.1 (AC_P)
- net at PS1.4 (DC+): now also CB1.1
- net GND: now reaches PS1.5 (DC-)
- net GND: now also PS2.5 (DC-), U1. (GND), U1.12 (GND), U1.23 (GND), J2.2 (Pin_2), SW2.4 (L), SW3.4 (L), U2.1 (GND)
- net at PS2.4 (DC+): now also CB1.3
- net Earth: now reaches P1.3 (EARTH)
- net +24V: now reaches U1.1 (VCC)
- net +24V: now also CB1.2, U2.5 (VBB)
- net PL1_DIR2: now reaches U1.10 (DIR2)
- net PL1_DIR2: now also U1.11 (DIR3), J3.26 (~{CE1}/GPIO7)
- net PL2_MEAS0: now reaches U1.13 (MEAS0)
- net PL2_MEAS0: now also J3.7 (GCLK0/GPIO4)
- net PL2_MEAS1: now reaches U1.14 (MEAS1)
- net PL2_MEAS1: now also J3.11 (GPIO17)
- net PL2_MEAS2: now reaches U1.15 (MEAS2)
- net PL2_MEAS2: now also J3.13 (GPIO27)
- net PL2_MEAS3: now reaches U1.16 (MEAS3)
- net PL2_MEAS3: now also J3.15 (GPIO22)
- net PL2_MEAS4: now reaches U1.17 (MEAS4)
- net PL2_MEAS4: now also J3.19 (MOSI0/GPIO10)
- net PL2_MEAS5: now reaches U1.18 (MEAS5)
- net PL2_MEAS5: now also J3.21 (MISO0/GPIO9)
- net PL2_MEAS6: now reaches U1.19 (MEAS6)
- net PL2_MEAS6: now also J3.23 (SCLK0/GPIO11), J3.36 (GPIO16)
- net +5V: now reaches U1.2 (VCTRL)
- net +5V: now also CB1.4, J2.1 (Pin_1), U2.4 (VREF)
- net PL2_MEAS7: now reaches U1.20 (MEAS7)
- net PL2_MEAS7: now also J3.38 (GPIO20/MOSI1)
- net PL3_PRINTER_ACTIVE: now reaches U1.21 (PWM0)
- net PL3_PRINTER_ACTIVE: now also J3.29 (GCLK1/GPIO5)
- net PL3_PRINTER_ANY0: now reaches U1.24 (ANY0)
- net PL3_PRINTER_ANY0: now also J3.31 (GCLK2/GPIO6)
- net PL3_PRINTER_ANY1: now reaches U1.25 (ANY1)
- net PL3_PRINTER_ANY1: now also J3.33 (PWM1/GPIO13)
- net PL3_PRINTER_ANY2: now reaches U1.26 (ANY2)
- net PL3_PRINTER_ANY2: now also J3.35 (GPIO19/MISO1)
- net LP_USER_HALT: now reaches U1.27 (ANY3)
- net LP_USER_HALT: now also U1.60 (T_ANY4), SW3.3 (L)
- net LP_USER_START: now reaches U1.28 (ANY4)
- net LP_USER_START: now also U1.59 (T_ANY3), J3.40 (GPIO21/SCLK1), SW2.3 (L)
- net PL1_EN: now reaches U1.3 (ENABLE)
- net PL1_EN: now also J3.8 (GPIO14/TXD)
- net at U1.33 (A1): now also M2.1
- net at U1.34 (AA1): now also M2.2 (-)
- net at U1.35 (B1): now also M2.3
- net at U1.36 (BB1): now also M2.4
- net at U1.37 (A2): now also M3.1
- net at U1.38 (AA2): now also M3.2 (-)
- net at U1.39 (B2): now also M3.3
- net PL1_STEP0: now reaches U1.4 (STEP0)
- net PL1_STEP0: now also J3.10 (GPIO15/RXD)
- net at U1.40 (BB2): now also M3.4
- net at U1.41 (A3): now also M4.1
- net at U1.42 (AA3): now also M4.2 (-)
- net at U1.43 (B3): now also M4.3
- net at U1.44 (BB3): now also M4.4
- net VMEAS: now reaches U1.45 (VMEAS)
- net VMEAS: now also SW2.1, SW3.1, SW4.2 (B), SW5.2 (B), SW6.2 (B), SW7.2 (B), SW8.2 (B), SW9.2 (B)
- net at U1.46 (SW0): now also SW4.1 (A)
- net at U1.47 (SW1): now also SW5.1 (A)
- net at U1.48 (SW2): now also SW7.1 (A)
- net at U1.49 (SW3): now also SW8.1 (A)
- net PL1_STEP1: now reaches U1.5 (STEP1)
- net PL1_STEP1: now also J3.12 (GPIO18/PWM0)
- net at U1.50 (SW4): now also SW9.1 (A)
- net SW_USER_START: now reaches U1.51 (SW5)
- net SW_USER_START: now also SW2.2
- net SW_USER_HALT: now reaches U1.52 (SW6)
- net SW_USER_HALT: now also SW3.2
- net at U1.53 (SW7): now also SW6.1 (A)
- net PRINTER_ANY0: now reaches U1.56 (T_ANY0)
- net PRINTER_ANY2: now reaches U1.57 (T_ANY2)
- net PRINTER_ANY1: now reaches U1.58 (T_ANY1)
- net PL1_STEP2: now reaches U1.6 (STEP2)
- net PL1_STEP2: now also U1.7 (STEP3), J3.16 (GPIO23)
- net PRINTER_GND: now reaches U1.61 (GND)
- net PRINTER_GND: now also U1.64 (GND)
- net PRINTER_ACTIVE: now reaches U1.62 (S_PWM0)
- net PRINTER_VCC: now reaches U1.63 (+5V)
- net PL1_DIR0: now reaches U1.8 (DIR0)
- net PL1_DIR0: now also J3.22 (GPIO25)
- net PL1_DIR1: now reaches U1.9 (DIR1)
- net PL1_DIR1: now also J3.24 (~{CE0}/GPIO8)
- new net: P1.1 (AC_P), SW1.2
- new net: P1.2 (AC_N), SW1.4
- new net: M5.1 (+), U2.6 (OUT1)
- new net: M5.2 (-), U2.8 (OUT2)
- new net MOT_PWM_1: J3.18 (GPIO24), U2.3 (IN1)
- new net MOT_PWM_2: J3.32 (PWM0/GPIO12), U2.2 (IN2)
- new net POW_5V: J1.1 (Pin_1), J3.4 (5V)
- new net POW_GND: J1.2 (Pin_2), J3.14 (GND), J3.20 (GND), J3.25 (GND), J3.30 (GND), J3.34 (GND), J3.39 (GND), J3.6 (GND), J3.9 (GND)
- no-connect marks 0 -> 12
Other:
- note added: "13/04/2023"
- note added: "Emergency halt"
- note added: "Main switch"
- note added: "Power plug"
- note added: "X - Axis"
- note added: "X' - Axis (fast)"
- note added: "Y - Axis"
- note added: "Z - Axis (1)"
- note added: "drake"
- note added: "drake electronics mk1"
- note added: "measurements"
- note added: "mk1.0.0"
- note added: "motors"
- note added: "power supply unit"
- note added: "printer tool"
- note added: "raspberry pi"
- note added: "user inputs"
- note added: "user interface"
- moved on the sheet: M1, P1, PS1, PS2

Commit message: updated electronics
Parts:
- removed CB1: CircuitBreaker_2P, symbol Device:CircuitBreaker_2P
- removed M5: Motor_DC, symbol Motor:Motor_DC
- removed SW2, SW3: SW_Push_Lamp, symbol Switch:SW_Push_Lamp
- removed SW4, SW5, SW6, SW7, SW8, SW9: SW_Push_Open, symbol Switch:SW_Push_Open
- removed U1: SYRD_MK1, symbol Driver_Motor:SYRD_MK1
- removed U2: A4950E, Package_SO:SOIC-8-1EP_3.9x4.9mm_P1.27mm_EP2.41x3.3mm, symbol Driver_Motor:A4950E
- added A1: Arduino_UNO_R2, Module:Arduino_UNO_R2, symbol MCU_Module:Arduino_UNO_R2
- added CB1: CircuitBreaker_3P, symbol Device:CircuitBreaker_3P
- added D1, D2, D3, D4, D5, D6: LED, symbol Device:LED
- added J10, J11, J12, J13, J14, J15, J16, J5, J6, J7, J8, J9: Conn_01x03, symbol Connector_Generic:Conn_01x03
- added J4: Conn_01x04, symbol Connector_Generic:Conn_01x04
- added J? (x4): USB_A, symbol Connector:USB_A
- added J?: Raspberry_Pi_2_3, symbol Connector:Raspberry_Pi_2_3
- added K?: DIPxx-2Axx-21x, Relay_THT:Relay_StandexMeder_DIP_LowProfile, symbol Relay:DIPxx-2Axx-21x
- added M10, M5, M6, M7, M8, M9: Motor_Servo, symbol Motor:Motor_Servo
- added P2: Conn_WallPlug_Earth, symbol Connector:Conn_WallPlug_Earth
- added PS3, PS4, PS5: VTX-214-015-124, Converter_ACDC:Converter_ACDC_Vigortronix_VTX-214-015-1xx_THT, symbol Converter_ACDC:VTX-214-015-124
- added R1, R10, R11, R12, R13, R14, R2, R3, R4, R5, R6, R7, R8, R9: R, symbol Device:R
- added SW2, SW3: SW_Push_LED, symbol Switch:SW_Push_LED
- added SW4, SW5, SW6, SW7, SW8, SW9: SW_Push_SPDT, symbol Switch:SW_Push_SPDT
- added SW?: SW_DPST, symbol Switch:SW_DPST
- added U1: SYRD_MK3, symbol syrd_mk3:SYRD_MK3
- added U2: LCD-016N002L, Display:LCD-016N002L, symbol Display_Character:LCD-016N002L
Connections:
- net PL3_PRINTER_ACTIVE is gone; now on net PL3_HEAD_1: J3.29 (GCLK1/GPIO5)
- net +24V: now also CB1.2, U1.1 (VCC)
- net +5V: now also J3.2 (5V), A1.8 (VIN), CB1.6, J?.1 (VBUS), J?.1 (VBUS), J?.1 (VBUS), SW2.1, SW3.1, U1.3 (+5V), U2.2 (VDD); no longer J2.1 (Pin_1)
- net Earth: now also P2.3 (EARTH)
- net GND: now also J3.39 (GND), A1.29 (GND), J?.4 (GND), J?.4 (GND), J?.4 (GND), J?.5 (Shield), J?.5 (Shield), J?.5 (Shield), PS3.5 (DC-), PS4.5 (DC-), SW2.3 (K), SW3.3 (K), U1.5 (GND), U1.59 (GND), U1.72 (GND), U2.1 (VSS); no longer J2.2 (Pin_2)
- net PL1_DIR0: now also U1.55 (DIR0)
- net PL1_DIR1: now also U1.56 (DIR1)
- net PL1_DIR2: now also U1.57 (DIR2), U1.58 (DIR3)
- net PL1_EN: now also U1.50 (ENABLE)
- net PL1_STEP0: now also U1.51 (STEP0)
- net PL1_STEP1: now also U1.52 (STEP1)
- net PL1_STEP2: now also U1.53 (STEP2), U1.54 (STEP3)
- net PL2_MEAS0: now also U1.60 (CONN0)
- net PL2_MEAS1: now also U1.61 (CONN1)
- net PL2_MEAS2: now also U1.62 (CONN2)
- net PL2_MEAS3: now also U1.63 (CONN3)
- net PL2_MEAS4: now also U1.64 (CONN4)
- net PL2_MEAS5: now also U1.65 (CONN5)
- net PL2_MEAS6: now also U1.66 (CONN6)
- net PL2_MEAS7: now also U1.67 (CONN7)
- net POW_GND: no longer J3.14 (GND), J3.20 (GND), J3.25 (GND), J3.30 (GND), J3.34 (GND), J3.39 (GND), J3.9 (GND)
- net at PS1.4 (DC+): now also CB1.1
- net at PS2.4 (DC+): now also CB1.3
- net at M1.1: now also U1.10 (A0)
- net at M1.2 (-): now also U1.11 (AA0)
- net at M1.3: now also U1.12 (B0)
- net at M1.4: now also U1.13 (BB0)
- net at PS1.2 (N), PS2.2 (N): now also K?.8, PS3.2 (N), PS4.2 (N); no longer SW1.3
- net at PS1.3 (L), PS2.3 (L): now also K?.7, PS3.3 (L), PS4.3 (L); no longer SW1.1
- net at M2.1: now also U1.20 (A1)
- net at M2.2 (-): now also U1.21 (AA1)
- net at M2.3: now also U1.22 (B1)
- net at M2.4: now also U1.23 (BB1)
- net at P1.1 (AC_P): now also SW?.2; no longer SW1.2
- net at P1.2 (AC_N): now also SW?.4; no longer SW1.4
- net PL3_HEAD_1: now reaches J3.37 (GPIO26)
- net PL3_HEAD_1: now also U1.70 (PWM0)
- net at M4.1: now also U1.40 (A3)
- net at M4.2 (-): now also U1.41 (AA3)
- net at M4.3: now also U1.42 (B3)
- net at M4.4: now also U1.43 (BB3)
- net at M3.1: now also U1.30 (A2)
- net at M3.2 (-): now also U1.31 (AA2)
- net at M3.3: now also U1.32 (B2)
- net at M3.4: now also U1.33 (BB2)
- net LP_USER_START renamed PL3_BED_SERVO4
- net PL3_BED_SERVO4: now also U1.76 (ANY3)
- net MOT_PWM_1 renamed PL1_STEP3
- net MOT_PWM_2 renamed PL1_DIR3
- net PL3_PRINTER_ANY0 renamed PL3_BED_SERVO1
- net PL3_BED_SERVO1: now also U1.73 (ANY0)
- net PL3_PRINTER_ANY1 renamed PL3_BED_SERVO2
- net PL3_BED_SERVO2: now also U1.74 (ANY1)
- net PL3_PRINTER_ANY2 renamed PL3_BED_SERVO3
- net PL3_BED_SERVO3: now also U1.75 (ANY2)
- new net: A1.9 (A0), SW2.2
- new net: R1.1, SW2.4 (A)
- new net: J8.1 (Pin_1), U1.140 (DEV8)
- new net: J8.2 (Pin_2), U1.141 (+5V)
- new net: J8.3 (Pin_3), U1.142 (GND)
- new net: A1.16 (D1/TX), J?.2 (D-)
- new net: A1.15 (D0/RX), J?.3 (D+)
- new net: J12.1 (Pin_1), R10.1, SW5.1 (A)
- new net: J12.2 (Pin_2), SW5.2 (B)
- new net: D2.1 (K), J12.3 (Pin_3), R10.2
- new net: J?.39 (GND), J?.4 (GND)
- new net: J?.1 (VBUS), J?.4 (5V)
- new net: CB1.5, PS3.4 (DC+)
- new net: K?.1, SW?.1
- new net: K?.14, SW?.3
- new net: M5.1 (PWM), U1.90 (S_PWM0)
- new net: M5.2 (+), U1.91 (+5V)
- new net: M5.3 (-), U1.92 (GND)
- new net: M10.1 (PWM), U1.115 (DEV3)
- new net: M10.2 (+), U1.116 (+5V)
- new net: M10.3 (-), U1.117 (GND)
- new net: D3.1 (K), J13.3 (Pin_3), R11.2
- new net: D3.2 (A), R5.2
- new net: J15.1 (Pin_1), R13.1, SW8.1 (A)
- new net: J15.2 (Pin_2), SW8.2 (B)
- new net: D5.1 (K), J15.3 (Pin_3), R13.2
- new net: J10.1 (Pin_1), U1.150 (DEV10)
- new net: J10.2 (Pin_2), U1.151 (+5V)
- new net: J10.3 (Pin_3), U1.152 (GND)
- new net: M7.1 (PWM), U1.100 (DEV0)
- new net: M7.2 (+), U1.101 (+5V)
- new net: M7.3 (-), U1.102 (GND)
- new net: D1.1 (K), J11.3 (Pin_3), R9.2
- new net: D1.2 (A), R3.2
- new net: R7.1, SW8.3 (C)
- new net: D6.1 (K), J16.3 (Pin_3), R14.2
- new net: D6.2 (A), R8.2
- new net: J13.1 (Pin_1), R11.1, SW6.1 (A)
- new net: J13.2 (Pin_2), SW6.2 (B)
- new net: R5.1, SW6.3 (C)
- new net: M8.1 (PWM), U1.105 (DEV1)
- new net: M8.2 (+), U1.106 (+5V)
- new net: M8.3 (-), U1.107 (GND)
- new net: M9.1 (PWM), U1.110 (DEV2)
- new net: M9.2 (+), U1.111 (+5V)
- new net: M9.3 (-), U1.112 (GND)
- new net: J5.1 (Pin_1), U1.125 (DEV5)
- new net: J5.2 (Pin_2), U1.126 (+5V)
- new net: J5.3 (Pin_3), U1.127 (GND)
- new net: J6.1 (Pin_1), U1.130 (DEV6)
- new net: J6.2 (Pin_2), U1.131 (+5V)
- new net: J6.3 (Pin_3), U1.132 (GND)
- new net: J7.1 (Pin_1), U1.135 (DEV7)
- new net: J7.2 (Pin_2), U1.136 (+5V)
- new net: J7.3 (Pin_3), U1.137 (GND)
- new net: J9.1 (Pin_1), U1.145 (DEV9)
- new net: J9.2 (Pin_2), U1.146 (+5V)
- new net: J9.3 (Pin_3), U1.147 (GND)
- new net: J4.1 (Pin_1), U1.185 (GND)
- new net: J4.2 (Pin_2), U1.186 (DEV5)
- new net: J4.3 (Pin_3), U1.187 (+5V)
- new net: J4.4 (Pin_4), U1.188 (GND)
- new net: M6.1 (PWM), U1.95 (S_PWM1)
- new net: M6.2 (+), U1.96 (+5V)
- new net: M6.3 (-), U1.97 (GND)
- new net: J14.1 (Pin_1), R12.1, SW7.1 (A)
- new net: J14.2 (Pin_2), SW7.2 (B)
- new net: D4.1 (K), J14.3 (Pin_3), R12.2
- new net: PS5.2 (N), SW1.3
- new net: PS5.3 (L), SW1.1
- new net: J2.1 (Pin_1), PS5.4 (DC+)
- new net: J2.2 (Pin_2), PS5.5 (DC-)
- new net: A1.10 (A1), R1.2
- new net: R6.1, SW7.3 (C)
- new net: D4.2 (A), R6.2
- new net: J16.1 (Pin_1), R14.1, SW9.1 (A)
- new net: J16.2 (Pin_2), SW9.2 (B)
- new net: P2.1 (AC_P), SW1.2
- new net: P2.2 (AC_N), SW1.4
- new net: R2.1, SW3.4 (A)
- new net: A1.12 (A3), R2.2
- new net: R8.1, SW9.3 (C)
- new net: R3.1, SW4.3 (C)
- new net: A1.11 (A2), SW3.2
- new net: J11.1 (Pin_1), R9.1, SW4.1 (A)
- new net: J11.2 (Pin_2), SW4.2 (B)
- new net: A1.18 (D3), U2.6 (E)
- new net: A1.19 (D4), U2.5 (R/~{W})
- new net: A1.20 (D5), U2.4 (RS)
- new net: A1.21 (D6), U2.7 (DB0)
- new net: A1.22 (D7), U2.8 (DB1)
- new net: A1.23 (D8), U2.9 (DB2)
- new net: A1.24 (D9), U2.10 (DB3)
- new net: A1.25 (D10), U2.11 (DB4)
- new net: A1.26 (D11), U2.12 (DB5)
- new net: A1.27 (D12), U2.13 (DB6)
- new net: A1.28 (D13), U2.14 (DB7)
- new net: R4.1, SW5.3 (C)
- new net: D2.2 (A), R4.2
- new net: D5.2 (A), R7.2
- new net +12V: CB1.4
- new net +3.3V: PS4.4 (DC+)
- new net PL3_HEAD_2: U1.71 (PWM1)
- new net RELAY_GND: A1.7 (GND), K?.6
- new net RELAY_IN: A1.14 (SCL/A5), K?.2
- no-connect marks 12 -> 49
Other:
- note added: "BL-TOUCH"
- note added: "Bed Motors"
- note added: "Head Motors"
- note added: "MEAS-X (1)"
- note added: "MEAS-X (2)"
- note added: "MEAS-Y (1)"
- note added: "MEAS-Y (2)"
- note added: "MEAS-Z (1)"
- note added: "MEAS-Z (2)"
- note added: "Z - Axis (2)"
- note added: "annotations"
- note added: "camera raspberry pi"
- note added: "drake robot"
- note added: "main power supply unit"
- note added: "main raspberry pi"
- note added: "output panel"
- note added: "standby power supply"
- note removed: "X' - Axis (fast)"
- note removed: "measurements"
- note removed: "power supply unit"
- note removed: "printer tool"
- note removed: "raspberry pi"
- note removed: "user inputs"
- note removed: "user interface"
- moved on the sheet: J1, J2, J3, M1, M2, M3, M4, P1, PS1, PS2, SW1
