File: electronics/drake_electronics/drake_electronics.kicad_sch (KiCad schematic)
At the start: 73 parts, among them J1 Conn_01x02_Female, J10 Conn_01x03, J11 Conn_01x03, J12 Conn_01x03, J13 Conn_01x03, J14 Conn_01x03, J15 Conn_01x03, J16 Conn_01x03, J2 Conn_01x02_Male, J3 Raspberry_Pi_2_3, J4 Conn_01x04, J5 Conn_01x03, J6 Conn_01x03, J7 Conn_01x03, J8 Conn_01x03, J9 Conn_01x03, M1 Stepper_Motor_bipolar, M10 Motor_Servo, M2 Stepper_Motor_bipolar, M3 Stepper_Motor_bipolar, M4 Stepper_Motor_bipolar, M5 Motor_Servo, M6 Motor_Servo, M7 Motor_Servo, M8 Motor_Servo, M9 Motor_Servo, P1 Conn_WallPlug_Earth, P2 Conn_WallPlug_Earth, SW1 SW_DPST, SW2 SW_Push_LED, SW3 SW_Push_LED, SW4 SW_Push_SPDT, SW5 SW_Push_SPDT, SW6 SW_Push_SPDT, SW7 SW_Push_SPDT, SW8 SW_Push_SPDT, SW9 SW_Push_SPDT, U1 SYRD_MK3, U2 LCD-016N002L

Commit message: updated electronics
Parts:
- removed A1: Arduino_UNO_R2, Module:Arduino_UNO_R2, symbol MCU_Module:Arduino_UNO_R2
- removed CB1: CircuitBreaker_3P, symbol Device:CircuitBreaker_3P
- removed J10, J11, J12, J13, J14, J15, J16, J5, J6, J7, J8, J9: Conn_01x03, symbol Connector_Generic:Conn_01x03
- removed J4: Conn_01x04, symbol Connector_Generic:Conn_01x04
- removed J? (x2): USB_A, symbol Connector:USB_A
- removed K?: DIPxx-2Axx-21x, Relay_THT:Relay_StandexMeder_DIP_LowProfile, symbol Relay:DIPxx-2Axx-21x
- removed M1, M2, M3, M4: Stepper_Motor_bipolar, symbol Motor:Stepper_Motor_bipolar
- removed M10, M9: Motor_Servo, symbol Motor:Motor_Servo
- removed R1, R2: R, symbol Device:R
- removed SW1, SW?: SW_DPST, symbol Switch:SW_DPST
- removed SW2, SW3: SW_Push_LED, symbol Switch:SW_Push_LED
- removed U1: SYRD_MK3, symbol syrd_mk3:SYRD_MK3
- removed U2: LCD-016N002L, Display:LCD-016N002L, symbol Display_Character:LCD-016N002L
- added J-BL, J-SC: Conn_01x05_Pin, symbol Connector:Conn_01x05_Pin
- added J-SC: Conn_01x05_Socket, symbol Connector:Conn_01x05_Socket
- added J-UT: J-UT, symbol Connector:Conn_01x06_Socket
- added J-UT: Conn_01x06_Pin, symbol Connector:Conn_01x06_Pin
- added J-X, J-Y, J-ZL, J-ZR: Conn_01x04_Pin, symbol Connector:Conn_01x04_Pin
- added J-X+, J-X-, J-Y+, J-Y-, J-Z+, J-Z-: Conn_01x03_Pin, symbol Connector:Conn_01x03_Pin
- added J-X+, J-X-, J-Y+, J-Y-, J-Z+, J-Z-: Conn_01x03_Socket, symbol Connector:Conn_01x03_Socket
- added J17, J29: Conn_01x05, symbol Connector_Generic:Conn_01x05
- added J18, J30: Conn_01x10, symbol Connector_Generic:Conn_01x10
- added J19, J20, J21, J23: Conn_01x04_Socket, symbol Connector:Conn_01x04_Socket
- added M1, M2, M3, M4: Motor_Servo, symbol Motor:Motor_Servo
- added M11, M12, M13, M14: Stepper_Motor_bipolar, symbol Motor:Stepper_Motor_bipolar
- added SW1, SW2: SW_MEC_5G_LED, symbol Switch:SW_MEC_5G_LED
- added U1, U2, U3, U4: STK672-080-E, symbol Driver_Motor:STK672-080-E
- J3: value Raspberry_Pi_2_3 -> Raspberry_Pi_3
- gave numbers to parts that had none: 3
Connections:
- net +12V: now also PS2.4 (DC+)
- net +24V: now also PS1.4 (DC+), J29.1 (Pin_1)
- net +3.3V: now also J3.17 (3V3), J-UT.1 (Pin_1), J-X+.2 (Pin_2), J-X-.2 (Pin_2), J-Y+.2 (Pin_2), J-Y-.2 (Pin_2), J-Z+.2 (Pin_2), J-Z-.2 (Pin_2), J17.5 (Pin_5), J29.5 (Pin_5)
- net +5V: now also M5.2 (+), M6.2 (+), M7.2 (+), M8.2 (+), PS3.4 (DC+), J-BL.1 (Pin_1), J-SC.1 (Pin_1), J-SC.1 (Pin_1), J17.4 (Pin_4), J29.2 (Pin_2), J29.4 (Pin_4), M1.2 (+), M2.2 (+), M3.2 (+), M4.2 (+)
- net GND: now also M5.3 (-), M6.3 (-), M7.3 (-), M8.3 (-), J-BL.3 (Pin_3), J-BL.5 (Pin_5), J-SC.5 (Pin_5), J-SC.5 (Pin_5), J-UT.6 (Pin_6), J-UT.6 (Pin_6), J-X+.3 (Pin_3), J-X-.3 (Pin_3), J-Y+.3 (Pin_3), J-Y-.3 (Pin_3), J-Z+.3 (Pin_3), J-Z-.3 (Pin_3), J17.3 (Pin_3), J18.10 (Pin_10), J29.3 (Pin_3), J30.10 (Pin_10), M1.3 (-), M2.3 (-), M3.3 (-), M4.3 (-), U1.1 (PG), U2.1 (PG), U2.12 (M3), U2.13 (~{RESET}), U2.8 (M1), U2.9 (M2), U3.1 (PG), U3.12 (M3), U3.13 (~{RESET}), U3.8 (M1), U3.9 (M2), U4.1 (PG), U4.12 (M3), U4.13 (~{RESET}), U4.8 (M1), U4.9 (M2)
- net at R10.1, SW5.1 (A): now also J-X-.1 (Pin_1)
- net at SW5.2 (B): now also J-X-.2 (Pin_2)
- net at D2.1 (K), R10.2: now also J-X-.3 (Pin_3)
- net at P1.1 (AC_P): now also PS1.3 (L), PS2.3 (L), PS3.3 (L), PS4.3 (L)
- net at P1.2 (AC_N): now also PS1.2 (N), PS2.2 (N), PS3.2 (N), PS4.2 (N)
- net ST_PWM5: now reaches M5.1 (PWM)
- net at D3.1 (K), R11.2: now also J-Y+.3 (Pin_3)
- net at R13.1, SW8.1 (A): now also J-Z+.1 (Pin_1)
- net at SW8.2 (B): now also J-Z+.2 (Pin_2)
- net at D5.1 (K), R13.2: now also J-Z+.3 (Pin_3)
- net ST_PWM7: now reaches M7.1 (PWM)
- net at D1.1 (K), R9.2: now also J-X+.3 (Pin_3)
- net at D6.1 (K), R14.2: now also J-Z-.3 (Pin_3)
- net at R11.1, SW6.1 (A): now also J-Y+.1 (Pin_1)
- net at SW6.2 (B): now also J-Y+.2 (Pin_2)
- net ST_PWM8: now reaches M8.1 (PWM)
- net ST_PWM6: now reaches M6.1 (PWM)
- net at R12.1, SW7.1 (A): now also J-Y-.1 (Pin_1)
- net at SW7.2 (B): now also J-Y-.2 (Pin_2)
- net at D4.1 (K), R12.2: now also J-Y-.3 (Pin_3)
- net at PS5.2 (N): now also P2.2 (AC_N)
- net at PS5.3 (L): now also P2.1 (AC_P)
- net at R14.1, SW9.1 (A): now also J-Z-.1 (Pin_1)
- net at SW9.2 (B): now also J-Z-.2 (Pin_2)
- net SC_SDA: now reaches J3.3 (SDA/GPIO2)
- net SC_SDA: now also J-SC.3 (Pin_3), J-SC.3 (Pin_3)
- net SC_SCL: now reaches J3.5 (SCL/GPIO3)
- net at R9.1, SW4.1 (A): now also J-X+.1 (Pin_1)
- net at SW4.2 (B): now also J-X+.2 (Pin_2)
- net PL1_DIR0: no longer names the net of J3.22 (GPIO25)
- net PL1_DIR1: no longer names the net of J3.24 (~{CE0}/GPIO8)
- net PL1_DIR2: no longer names the net of J3.26 (~{CE1}/GPIO7)
- net PL1_DIR3 renamed STEP_X
- net STEP_X: now also J30.2 (Pin_2)
- net PL1_EN: no longer names the net of J3.8 (GPIO14/TXD)
- net PL1_STEP0: no longer names the net of J3.10 (GPIO15/RXD)
- net PL1_STEP1: no longer names the net of J3.12 (GPIO18/PWM0)
- net PL1_STEP2: no longer names the net of J3.16 (GPIO23)
- net PL1_STEP3: no longer names the net of J3.18 (GPIO24)
- net PL2_MEAS0 renamed BL_MEAS
- net BL_MEAS: now also J-BL.4 (Pin_4)
- net PL2_MEAS1: no longer names the net of J3.11 (GPIO17)
- net PL2_MEAS2: no longer names the net of J3.13 (GPIO27)
- net PL2_MEAS3: no longer names the net of J3.15 (GPIO22)
- net PL2_MEAS4: no longer names the net of J3.19 (MOSI0/GPIO10)
- net PL2_MEAS5: no longer names the net of J3.21 (MISO0/GPIO9)
- net PL2_MEAS6: no longer names the net of J3.23 (SCLK0/GPIO11)
- net PL2_MEAS6: no longer J3.36 (GPIO16)
- net PL2_MEAS7 renamed STEP_Y
- net STEP_Y: now also J30.3 (Pin_3)
- net PL3_BED_SERVO1 renamed MEAS_Y+
- net MEAS_Y+: now also J-Y+.1 (Pin_1)
- net PL3_BED_SERVO2 renamed DIR_Y
- net DIR_Y: now also J30.7 (Pin_7)
- net PL3_BED_SERVO3: no longer names the net of J3.35 (GPIO19/MISO1)
- net PL3_BED_SERVO4 renamed DIR_X
- net DIR_X: now also J30.6 (Pin_6)
- net PL3_HEAD_1: no longer names the net of J3.37 (GPIO26)
- net PL3_HEAD_1: no longer J3.29 (GCLK1/GPIO5)
- new net: J-Y.1 (Pin_1), U2.5 (A)
- new net: J-Y.2 (Pin_2), U2.4 (AB)
- new net: J-Y.3 (Pin_3), U2.3 (B)
- new net: J-Y.4 (Pin_4), U2.2 (BB)
- new net: J-UT.1 (Pin_1), SW1.3 (K), SW1.4 (A), SW2.3 (K), SW2.4 (A)
- new net: J-UT.2 (Pin_2), SW1.1
- new net: J-UT.3 (Pin_3), SW1.2
- new net: J-UT.4 (Pin_4), SW2.1
- new net: J-UT.5 (Pin_5), SW2.2
- new net: J-X.1 (Pin_1), U1.5 (A)
- new net: J-X.2 (Pin_2), U1.4 (AB)
- new net: J-X.3 (Pin_3), U1.3 (B)
- new net: J-X.4 (Pin_4), U1.2 (BB)
- new net: J-ZL.1 (Pin_1), U3.5 (A)
- new net: J-ZL.2 (Pin_2), U3.4 (AB)
- new net: J-ZL.3 (Pin_3), U3.3 (B)
- new net: J-ZL.4 (Pin_4), U3.2 (BB)
- new net: J21.1 (Pin_1), M13.1
- new net: J21.2 (Pin_2), M13.2 (-)
- new net: J21.3 (Pin_3), M13.3
- new net: J21.4 (Pin_4), M13.4
- new net: J18.7 (Pin_7), U2.10 (CWB)
- new net: J18.4 (Pin_4), U3.11 (CLOCK)
- new net: J18.5 (Pin_5), U4.11 (CLOCK)
- new net: J18.6 (Pin_6), U1.10 (CWB)
- new net: J18.8 (Pin_8), U3.10 (CWB)
- new net: J18.9 (Pin_9), U4.10 (CWB)
- new net: J19.1 (Pin_1), M11.1
- new net: J19.2 (Pin_2), M11.2 (-)
- new net: J19.3 (Pin_3), M11.3
- new net: J19.4 (Pin_4), M11.4
- new net: J-ZR.1 (Pin_1), U4.5 (A)
- new net: J-ZR.2 (Pin_2), U4.4 (AB)
- new net: J-ZR.3 (Pin_3), U4.3 (B)
- new net: J-ZR.4 (Pin_4), U4.2 (BB)
- new net: J23.1 (Pin_1), M14.1
- new net: J23.2 (Pin_2), M14.2 (-)
- new net: J23.3 (Pin_3), M14.3
- new net: J23.4 (Pin_4), M14.4
- new net: J20.1 (Pin_1), M12.1
- new net: J20.2 (Pin_2), M12.2 (-)
- new net: J20.3 (Pin_3), M12.3
- new net: J20.4 (Pin_4), M12.4
- new net BL_ACT: J-BL.2 (Pin_2)
- new net DIR_Z: J30.8 (Pin_8), J30.9 (Pin_9)
- new net ENABLE: J18.1 (Pin_1), J30.1 (Pin_1), U1.15 (ENABLE), U2.15 (ENABLE), U3.15 (ENABLE), U4.15 (ENABLE)
- new net MEAS_X+: J-X+.1 (Pin_1), J3.29 (GCLK1/GPIO5)
- new net MEAS_X-: J-X-.1 (Pin_1)
- new net MEAS_Y-: J-Y-.1 (Pin_1)
- new net MEAS_Z+: J-Z+.1 (Pin_1)
- new net MEAS_Z-: J-Z-.1 (Pin_1)
- new net PWM: J18.2 (Pin_2), J18.3 (Pin_3), U1.11 (CLOCK), U2.11 (CLOCK)
- new net SC_CLK: J-SC.4 (Pin_4), J-SC.4 (Pin_4)
- new net SC_VCC: J-SC.2 (Pin_2), J-SC.2 (Pin_2)
- new net STEP_Z: J30.4 (Pin_4), J30.5 (Pin_5)
- new net ST_PWM1: M1.1 (PWM)
- new net ST_PWM2: M2.1 (PWM)
- new net ST_PWM3: M3.1 (PWM)
- new net ST_PWM4: M4.1 (PWM)
- new net UT_LED_HALT: J-UT.5 (Pin_5)
- new net UT_LED_START: J-UT.3 (Pin_3)
- new net UT_SW_HALT: J-UT.4 (Pin_4)
- new net UT_SW_START: J-UT.2 (Pin_2)
- new net VCC: J17.1 (Pin_1), U1.12 (M3), U1.13 (~{RESET}), U1.6 (VCC), U1.8 (M1), U1.9 (M2), U2.6 (VCC), U3.6 (VCC), U4.6 (VCC)
- new net VCTRL: J17.2 (Pin_2), U1.7 (Vref), U2.7 (Vref), U3.7 (Vref), U4.7 (Vref)
- no-connect marks 49 -> 17
Other:
- note added: "MEAS-NEG-X"
- note added: "MEAS-NEG-Y"
- note added: "MEAS-NEG-Z"
- note added: "MEAS-POS-X"
- note added: "MEAS-POS-Y"
- note added: "MEAS-POS-Z"
- note added: "PSC"
- note added: "Servo Table and Controller (SC)"
- note added: "User terminal (UT)"
- note added: "driver unit"
- note added: "mk1.1.0"
- note added: "motors (external)"
- note removed: "BL-TOUCH"
- note removed: "Bed Motors"
- note removed: "Emergency halt"
- note removed: "Head Motors"
- note removed: "MEAS-X (1)"
- note removed: "MEAS-X (2)"
- note removed: "MEAS-Y (1)"
- note removed: "MEAS-Y (2)"
- note removed: "MEAS-Z (1)"
- note removed: "MEAS-Z (2)"
- note removed: "Main switch"
- note removed: "X - Axis"
- note removed: "Y - Axis"
- note removed: "Z - Axis (1)"
- note removed: "Z - Axis (2)"
- note removed: "drake robot"
- note removed: "mk1.0.0"
- note removed: "motors"
- note removed: "output panel"
- moved on the sheet: J27, J28, J3, J4, P2, PS1, PS2, PS3, PS4, SW4, SW5, SW6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
